Commit message: Task 6

File: task5/ex05/install/robot_description/share/robot_description/urdf/gazebo.urdf.xacro (robot description, xacro)
@@ -13,5 +13,9 @@
       <wheel_radius>0.033</wheel_radius>
       <odom_publish_frequency>10</odom_publish_frequency>
-      <topic>cmd_vel</topic>
+      <topic>/model/robot/cmd_vel</topic>
+      <min_velocity>-1.0</min_velocity>
+      <max_velocity>1.0</max_velocity>
+      <min_acceleration>-1.0</min_acceleration>
+      <max_acceleration>1.0</max_acceleration>
     </plugin>
     <plugin filename="gz-sim-odometry-publisher-system" name="gz::sim::systems::OdometryPublisher">

File: task5/ex05/install/robot_description/share/robot_description/urdf/robot.urdf.xacro (robot description, xacro)
@@ -12,8 +12,12 @@
   <xacro:property name="rear_wheel_offset_x" value="-0.113"/>
   <xacro:property name="wheel_offset_y" value="0.1485"/>
-  <xacro:property name="caster_wheel_radius" value="0.01"/>
-  <xacro:property name="caster_wheel_mass" value="0.01"/>
-  <xacro:property name="caster_wheel_offset_x" value="0.075"/>
   <xacro:property name="mass" value="1.0"/>
+  <!-- New properties for steam locomotive elements -->
+  <xacro:property name="pipe_radius" value="${chassis_width/4}"/>
+  <xacro:property name="pipe_height" value="0.15"/>
+  <xacro:property name="cabin_wall_thickness" value="0.015"/>
+  <xacro:property name="cabin_wall_height" value="0.08"/>
+  <xacro:property name="cabin_roof_thickness" value="0.02"/>
+  <xacro:property name="cabin_length" value="${chassis_length/3}"/>
   <!-- Materials -->
   <material name="white">
@@ -32,4 +36,13 @@
     <color rgba="1 0 0 1"/>
   </material>
+  <material name="gray">
+    <color rgba="0.5 0.5 0.5 1"/>
+  </material>
+  <material name="dark_gray">
+    <color rgba="0.3 0.3 0.3 1"/>
+  </material>
+  <material name="glass">
+    <color rgba="0.7 0.9 1.0 0.6"/>
+  </material>
   <!-- Main chassis link that contains the robot body -->
   <link name="base_link">
@@ -70,4 +83,150 @@
     <origin xyz="0 0 -${chassis_height/2}" rpy="0 0 0"/>
   </joint>
+  <!-- Steam Pipe (moved closer to cabin, front edge aligned with chassis front) -->
+  <link name="steam_pipe">
+    <inertial>
+      <origin xyz="0 0 ${pipe_height/2}" rpy="0 0 0"/>
+      <mass value="0.1"/>
+      <inertia
+        ixx="${(1/12) * 0.1 * (3*pipe_radius*pipe_radius + pipe_height*pipe_height)}"
+        ixy="0.0"
+        ixz="0.0"
+        iyy="${(1/12) * 0.1 * (3*pipe_radius*pipe_radius + pipe_height*pipe_height)}"
+        iyz="0.0"
+        izz="${(1/2) * 0.1 * (pipe_radius*pipe_radius)}"
+      />
+    </inertial>
+    <visual>
+      <origin xyz="0 0 ${pipe_height/2}"/>
+      <geometry>
+        <cylinder radius="${pipe_radius}" length="${pipe_height}"/>
+      </geometry>
+      <material name="dark_gray"/>
+    </visual>
+    <collision>
+      <origin xyz="0 0 ${pipe_height/2}"/>
+      <geometry>
+        <cylinder radius="${pipe_radius}" length="${pipe_height}"/>
+      </geometry>
+    </collision>
+  </link>
+  <joint name="steam_pipe_joint" type="fixed">
+    <parent link="base_link"/>
+    <child link="steam_pipe"/>
+    <origin xyz="${chassis_length/2 - pipe_radius} 0 ${chassis_height}" rpy="0 0 0"/>
+  </joint>
+  <gazebo reference="steam_pipe">
+    <material>Gazebo/DarkGray</material>
+  </gazebo>
+  <!-- Cabin Left Wall (full width at the edges) -->
+  <link name="cabin_left_wall">
+    <inertial>
+      <origin xyz="0 0 ${cabin_wall_height/2}" rpy="0 0 0"/>
+      <mass value="0.05"/>
+      <inertia
+        ixx="${(1/12) * 0.05 * (cabin_wall_thickness*cabin_wall_thickness + cabin_wall_height*cabin_wall_height)}"
+        ixy="0.0"
+        ixz="0.0"
+        iyy="${(1/12) * 0.05 * (cabin_length*cabin_length + cabin_wall_height*cabin_wall_height)}"
+        iyz="0.0"
+        izz="${(1/12) * 0.05 * (cabin_length*cabin_length + cabin_wall_thickness*cabin_wall_thickness)}"
+      />
+    </inertial>
+    <visual>
+      <origin xyz="0 0 ${cabin_wall_height/2}"/>
+      <geometry>
+        <box size="${cabin_length} ${cabin_wall_thickness} ${cabin_wall_height}"/>
+      </geometry>
+      <material name="glass"/>
+    </visual>
+    <collision>
+      <origin xyz="0 0 ${cabin_wall_height/2}"/>
+      <geometry>
+        <box size="${cabin_length} ${cabin_wall_thickness} ${cabin_wall_height}"/>
+      </geometry>
+    </collision>
+  </link>
+  <joint name="cabin_left_wall_joint" type="fixed">
+    <parent link="base_link"/>
+    <child link="cabin_left_wall"/>
+    <origin xyz="${-chassis_length/3} ${chassis_width/2 - cabin_wall_thickness/2} ${chassis_height}" rpy="0 0 0"/>
+  </joint>
+  <gazebo reference="cabin_left_wall">
+    <material>Gazebo/Blue</material>
+  </gazebo>
+  <!-- Cabin Right Wall (full width at the edges) -->
+  <link name="cabin_right_wall">
+    <inertial>
+      <origin xyz="0 0 ${cabin_wall_height/2}" rpy="0 0 0"/>
+      <mass value="0.05"/>
+      <inertia
+        ixx="${(1/12) * 0.05 * (cabin_wall_thickness*cabin_wall_thickness + cabin_wall_height*cabin_wall_height)}"
+        ixy="0.0"
+        ixz="0.0"
+        iyy="${(1/12) * 0.05 * (cabin_length*cabin_length + cabin_wall_height*cabin_wall_height)}"
+        iyz="0.0"
+        izz="${(1/12) * 0.05 * (cabin_length*cabin_length + cabin_wall_thickness*cabin_wall_thickness)}"
+      />
+    </inertial>
+    <visual>
+      <origin xyz="0 0 ${cabin_wall_height/2}"/>
+      <geometry>
+        <box size="${cabin_length} ${cabin_wall_thickness} ${cabin_wall_height}"/>
+      </geometry>
+      <material name="glass"/>
+    </visual>
+    <collision>
+      <origin xyz="0 0 ${cabin_wall_height/2}"/>
+      <geometry>
+        <box size="${cabin_length} ${cabin_wall_thickness} ${cabin_wall_height}"/>
+      </geometry>
+    </collision>
+  </link>
+  <joint name="cabin_right_wall_joint" type="fixed">
+    <parent link="base_link"/>
+    <child link="cabin_right_wall"/>
+    <origin xyz="${-chassis_length/3} ${-chassis_width/2 + cabin_wall_thickness/2} ${chassis_height}" rpy="0 0 0"/>
+  </joint>
+  <gazebo reference="cabin_right_wall">
+    <material>Gazebo/Blue</material>
+  </gazebo>
+  <!-- Cabin Roof (full width of chassis, touching the walls) -->
+  <link name="cabin_roof">
+    <inertial>
+      <origin xyz="0 0 ${cabin_roof_thickness/2}" rpy="0 0 0"/>
+      <mass value="0.1"/>
+      <inertia
+        ixx="${(1/12) * 0.1 * (cabin_roof_thickness*cabin_roof_thickness + chassis_width*chassis_width)}"
+        ixy="0.0"
+        ixz="0.0"
+        iyy="${(1/12) * 0.1 * (cabin_length*cabin_length + chassis_width*chassis_width)}"
+        iyz="0.0"
+        izz="${(1/12) * 0.1 * (cabin_length*cabin_length + cabin_roof_thickness*cabin_roof_thickness)}"
+      />
+    </inertial>
+    <visual>
+      <origin xyz="0 0 ${cabin_roof_thickness/2}"/>
+      <geometry>
+        <box size="${cabin_length} ${chassis_width} ${cabin_roof_thickness}"/>
+      </geometry>
+      <material name="gray"/>
+    </visual>
+    <collision>
+      <origin xyz="0 0 ${cabin_roof_thickness/2}"/>
+      <geometry>
+        <box size="${cabin_length} ${chassis_width} ${cabin_roof_thickness}"/>
+      </geometry>
+    </collision>
+  </link>
+  <joint name="cabin_roof_joint" type="fixed">
+    <parent link="base_link"/>
+    <child link="cabin_roof"/>
+    <!-- Adjusted to ensure roof touches the walls -->
+    <origin xyz="${-chassis_length/3} 0 ${chassis_height + cabin_wall_height}" rpy="0 0 0"/>
+  </joint>
+  <gazebo reference="cabin_roof">
+    <material>Gazebo/Gray</material>
+  </gazebo>
+  <!-- Wheels (unchanged) -->
   <!-- Front Left Wheel -->
   <joint name="front_left_wheel_joint" type="continuous">
@@ -218,39 +377,3 @@
     <material>Gazebo/Blue</material>
   </gazebo>
-  <!-- Caster Wheel -->
-  <joint name="caster_wheel_joint" type="fixed">
-    <parent link="base_link"/>
-    <child link="caster_wheel"/>
-    <origin xyz="${caster_wheel_offset_x} 0 -${chassis_height/2 + caster_wheel_radius}"/>
-  </joint>
-  <link name="caster_wheel">
-    <visual>
-      <geometry>
-        <sphere radius="${caster_wheel_radius}"/>
-      </geometry>
-      <material name="white"/>
-    </visual>
-    <collision>
-      <geometry>
-        <sphere radius="${caster_wheel_radius}"/>
-      </geometry>
-    </collision>
-    <inertial>
-      <origin xyz="0 0 0" rpy="0 0 0"/>
-      <mass value="${caster_wheel_mass}" />
-      <inertia
-        ixx="${(2/5) * caster_wheel_mass * (caster_wheel_radius*caster_wheel_radius)}"
-        ixy="0.0"
-        ixz="0.0"
-        iyy="${(2/5) * caster_wheel_mass * (caster_wheel_radius*caster_wheel_radius)}"
-        iyz="0.0"
-        izz="${(2/5) * caster_wheel_mass * (caster_wheel_radius*caster_wheel_radius)}"
-      />
-    </inertial>
-  </link>
-  <gazebo reference="caster_wheel">
-    <material>Gazebo/White</material>
-    <mu1 value="0.001"/>
-    <mu2 value="0.001"/>
-  </gazebo>
 </robot>
